File: LS_2026_vyuka/jvc/vodotrysk/control_board/control_board.kicad_sch (KiCad schematic)
At the start: 74 parts, among them J1 PWR_IN, J10 WS2812B, J11 WS2812B_PWR, J12 CONN_PUMP1, J13 USB_C, J2 DATA_OUT, J3 DC jack in, J4 PWR_OUT, J5 CONN_PUMP1, J6 WATER_LEVEL_1, J7 WATER_LEVEL_2, J8 I2C, J9 UART, SW1 BTN_RST, SW2 BTN_BOOT0, U1 ESP32-S3-WROOM-1-N4, U2 AHT20, U3 AMS1117-3.3, U4 INA180A2, U5 TPS5430DDA, U6 DS3231MZ

Commit message: latest update
Parts:
- added R?: 5k1, Resistor_SMD:R_0805_2012Metric, symbol Device:R
Connections:
- net +3.3V: now also R?.1
- net BOOT0: now also R?.2
- net SW_PUMP1: now also U1.8 (IO15); no longer U1.26 (IO45)
Changed lines of the file:
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@@
 	)
 	(junction
+		(at 218.44 34.29)
+		(diameter 0)
+		(color 0 0 0 0)
+	)
+	(junction
 		(at 241.3 151.13)
 		(diameter 0)
@@
 	(wire
 		(pts
+			(xy 218.44 34.29) (xy 219.71 34.29)
+		)
+		(stroke
+			(width 0)
+			(type default)
+		)
+	)
+	(wire
+		(pts
 			(xy 29.21 74.93) (xy 39.37 74.93)
 		)
@@
 	(wire
 		(pts
+			(xy 217.17 34.29) (xy 218.44 34.29)
+		)
+		(stroke
+			(width 0)
+			(type default)
+		)
+	)
+	(wire
+		(pts
 			(xy 240.03 66.04) (xy 247.65 66.04)
 		)
@@
 	(wire
 		(pts
-			(xy 218.44 34.29) (xy 219.71 34.29)
-		)
-		(stroke
-			(width 0)
-			(type default)
-		)
-	)
-	(wire
-		(pts
 			(xy 36.83 72.39) (xy 39.37 72.39)
 		)
@@
 		)
 	)
+	(global_label "SW_PUMP1"
+		(shape input)
+		(at 210.82 143.51 180)
+		(fields_autoplaced yes)
+		(effects
+			(font
+				(size 1.27 1.27)
+			)
+			(justify right)
+		)
+		(property "Intersheetrefs" "${INTERSHEET_REFS}"
+			(at 197.6749 143.51 0)
+			(effects
+				(font
+					(size 1.27 1.27)
+				)
+				(justify right)
+				(hide yes)
+			)
+		)
+	)
 	(global_label "CURR_ADC2"
 		(shape input)
@@
 		)
 	)
-	(global_label "SW_PUMP1"
-		(shape input)
-		(at 241.3 138.43 0)
-		(fields_autoplaced yes)
-		(effects
-			(font
-				(size 1.27 1.27)
-			)
-			(justify left)
-		)
-		(property "Intersheetrefs" "${INTERSHEET_REFS}"
-			(at 254.4451 138.43 0)
-			(effects
-				(font
-					(size 1.27 1.27)
-				)
-				(justify left)
-				(hide yes)
-			)
-		)
-	)
 	(global_label "WS2812B"
 		(shape input)
@@
 	(global_label "BOOT0"
 		(shape input)
-		(at 218.44 34.29 180)
+		(at 217.17 34.29 180)
 		(fields_autoplaced yes)
 		(effects
@@
 		)
 		(property "Intersheetrefs" "${INTERSHEET_REFS}"
-			(at 209.3467 34.29 0)
+			(at 208.0767 34.29 0)
 			(effects
 				(font
@@
 		(on_board yes)
 		(dnp no)
-		(fields_autoplaced yes)
 		(property "Reference" "SW2"
-			(at 224.79 26.67 0)
+			(at 230.886 29.21 0)
 			(effects
 				(font
@@
 		)
 		(property "Value" "BTN_BOOT0"
-			(at 224.79 29.21 0)
+			(at 230.886 31.75 0)
 			(effects
 				(font
@@
 	)
 	(symbol
+		(lib_id "power:+3.3V")
+		(at 218.44 26.67 0)
+		(unit 1)
+		(exclude_from_sim no)
+		(in_bom yes)
+		(on_board yes)
+		(dnp no)
+		(fields_autoplaced yes)
+		(property "Reference" "#PWR082"
+			(at 218.44 30.48 0)
+			(effects
+				(font
+					(size 1.27 1.27)
+				)
+				(hide yes)
+			)
+		)
+		(property "Value" "+3.3V"
+			(at 218.44 21.59 0)
+			(effects
+				(font
+					(size 1.27 1.27)
+				)
+			)
+		)
+		(property "Footprint" ""
+			(at 218.44 26.67 0)
+			(effects
+				(font
+					(size 1.27 1.27)
+				)
+				(hide yes)
+			)
+		)
+		(property "Datasheet" ""
+			(at 218.44 26.67 0)
+			(effects
+				(font
+					(size 1.27 1.27)
+				)
+				(hide yes)
+			)
+		)
+		(property "Description" "Power symbol creates a global label with name \"+3.3V\""
+			(at 218.44 26.67 0)
+			(effects
+				(font
+					(size 1.27 1.27)
+				)
+				(hide yes)
+			)
+		)
+		(pin "1"
+		)
+		(instances
+			(project "control_board"
+				(path "/929a66e8-f002-4a52-9495-2c08f5a001e7"
+					(reference "#PWR082")
+					(unit 1)
+				)
+			)
+		)
+	)
+	(symbol
 		(lib_id "Device:R")
 		(at 194.31 62.23 0)
@@
 					(unit 1)
 				)
+			)
+		)
+	)
+	(symbol
+		(lib_id "Device:R")
+		(at 218.44 30.48 0)
+		(unit 1)
+		(exclude_from_sim no)
+		(in_bom yes)
+		(on_board yes)
+		(dnp no)
+		(property "Reference" "R?"
+			(at 212.09 28.956 0)
+			(effects
+				(font
+					(size 1.27 1.27)
+				)
+				(justify left)
+			)
+		)
+		(property "Value" "5k1"
+			(at 212.09 31.496 0)
+			(effects
+				(font
+					(size 1.27 1.27)
+				)
+				(justify left)
+			)
+		)
+		(property "Footprint" "Resistor_SMD:R_0805_2012Metric"
+			(at 216.662 30.48 90)
+			(effects
+				(font
+					(size 1.27 1.27)
+				)
+				(hide yes)
+			)
+		)
+		(property "Datasheet" "~"
+			(at 218.44 30.48 0)
+			(effects
+				(font
+					(size 1.27 1.27)
+				)
+				(hide yes)
+			)
+		)
+		(property "Description" "Resistor"
+			(at 218.44 30.48 0)
+			(effects
+				(font
+					(size 1.27 1.27)
+				)
+				(hide yes)
+			)
+		)
+		(property "LCSC" "C27834"
+			(at 218.44 30.48 0)
+			(effects
+				(font
+					(size 1.27 1.27)
+				)
+				(hide yes)
+			)
+		)
+		(pin "2"
+		)
+		(pin "1"
+		)
+		(instances
+			(project "control_board"
+				(path "/929a66e8-f002-4a52-9495-2c08f5a001e7"
+					(reference "R?")
+					(unit 1)
+				)
